File: _autosave-power board.kicad_pcb (KiCad board)
At the start: 2 copper layers, 63.5 x 90.8 mm, 36 parts, among them J1 Conn_01x02_Female, J11 Conn_01x02_Female, J12 Conn_01x02_Female, J2 Conn_01x02_Female, J3 Conn_01x02_Female, J4 Conn_01x02_Female, J5 Conn_01x02_Female, J6 Conn_01x02_Female, J7 Conn_01x02_Female, J8 Conn_01x02_Female, J9 Conn_01x02_Female, Q1 STP160N3LL, U1 THL-25-2411

Commit message: updated board to v1.2
Parts:
- removed H21, H22: MountingHole_Pad, TestPoint:TestPoint_THTPad_D3.0mm_Drill1.5mm
- added C10: 3UF, Capacitor_SMD:C_0805_2012Metric_Pad1.15x1.40mm_HandSolder, F.Cu at (43.9, 99.3)
- added C11: 3UF, Capacitor_SMD:C_0805_2012Metric_Pad1.15x1.40mm_HandSolder, F.Cu at (67.0, 43.8)
- added C12: 3UF, Capacitor_SMD:C_0805_2012Metric_Pad1.15x1.40mm_HandSolder, F.Cu at (76.0, 58.4)
- added C4: 470UF, Capacitor_THT:CP_Radial_D10.0mm_P5.00mm, F.Cu at (38.1, 55.2)
- added C7: 470UF, Capacitor_THT:CP_Radial_D10.0mm_P5.00mm, F.Cu at (44.5, 79.4)
- added J10: Barrel_Jack, Connector_BarrelJack:BarrelJack_CUI_PJ-063AH_Horizontal, F.Cu at (71.9, 50.5)
- added Q2: STP160N3LL, kicad-footprints-master:MOSFET_Down, F.Cu at (59.3, 91.7)
- added R7: R, Resistor_SMD:R_0805_2012Metric_Pad1.15x1.40mm_HandSolder, F.Cu at (38.1, 74.0)
- added R8: R, Resistor_SMD:R_0805_2012Metric_Pad1.15x1.40mm_HandSolder, F.Cu at (50.4, 51.4)
- H1, H2, H3, H4: footprint MountingHole:MountingHole_3.2mm_M3 -> MountingHole:MountingHole_3.2mm_M3_Pad_Via
- Q1: footprint TO254P1040X460X1935-3:TO254P1040X460X1935-3 -> kicad-footprints-master:MOSFET_Down
- moved C3 52.8 mm to (40.6, 44.5)
- moved J7 29.2 mm to (68.4, 36.3)
- moved S1 28.1 mm to (43.4, 105.2)
- moved J9 25.3 mm to (30.3, 109.3)
- moved J8 23.6 mm to (30.1, 46.2)
- moved R2 21.7 mm to (37.8, 97.3), turned to 90 degrees
- moved C8 18.9 mm to (56.5, 45.1), turned to 180 degrees
- moved R1 16.4 mm to (37.7, 101.8)
- moved C1 14.9 mm to (41.2, 97.3), turned to 90 degrees
- moved Q1 10.8 mm to (59.4, 104.1)
- moved J6 9.35 mm to (49.3, 111.3)
- moved D2 7.43 mm to (68.4, 54.7), turned to 90 degrees
- moved C6 5.75 mm to (44.5, 90.2)
- moved H4 4.56 mm to (79.4, 38.2)
- moved C5 3.99 mm to (44.5, 67.8)
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Connections:
- net Net-(Q1-Pad2) renamed /gate
- C3 pad 2: safe-V24 -> GND
- C8 pad 2: safe-V24 -> GND
- D1 pad 1: GND -> safe-V24
- S1 pad 3: GND -> Net-(C10-Pad2)
Routing:
- net +24V: track 22.8 -> 67.4 mm, vias 4 -> 0
- net ISO_GND_5V: track 18.3 -> 31.7 mm
- net /gate: track 16.4 -> 29.8 mm
- net Net-(C12-Pad2): track 0.00 -> 11.0 mm
- net safe-V24: track 0.00 -> 10.8 mm
- net GND: track 136.0 -> 146.8 mm, vias 5 -> 2
- net Net-(C1-Pad1): track 22.2 -> 13.5 mm, vias 1 -> 0
- net Net-(C10-Pad2): track 0.00 -> 7.40 mm
- net Net-(D2-Pad2): track 4.60 -> 2.91 mm
- net Net-(L1-Pad2): track 34.9 -> 34.3 mm, vias 0 -> 1
- added copper zone on B.Cu, net +24V
- added copper zone on F.Cu, net safe-V24
- removed copper zone on F.Cu, net +24V
- removed copper zone on B.Cu, net safe-V24
Other:
- board text removed: "ISO_5V"
- board text removed: "ISO_GND"
- board text removed: "XT30 x 7"
