File: power board.sch (KiCad schematic (older format))
At the start: 38 parts, among them J1 Conn_01x02_Female, J11 Conn_01x02_Female, J12 Conn_01x02_Female, J2 Conn_01x02_Female, J3 Conn_01x02_Female, J4 Conn_01x02_Female, J5 Conn_01x02_Female, J6 Conn_01x02_Female, J7 Conn_01x02_Female, J8 Conn_01x02_Female, J9 Conn_01x02_Female, Q1 STP160N3LL, U1 THL-25-2411

Commit message: updated board to v1.2
Parts:
- removed H21, H22: MountingHole_Pad, TestPoint:TestPoint_THTPad_D3.0mm_Drill1.5mm, symbol Mechanical:MountingHole_Pad
- added C10, C11, C12: 3UF, Capacitor_SMD:C_0805_2012Metric_Pad1.15x1.40mm_HandSolder, symbol Device:C
- added J10: Barrel_Jack, Connector_BarrelJack:BarrelJack_CUI_PJ-063AH_Horizontal, symbol Connector:Barrel_Jack
- added Q2: STP160N3LL, kicad-footprints-master:MOSFET_Down, symbol Transistor_FET:IRF6711S
- added R7: R, Resistor_SMD:R_0805_2012Metric_Pad1.15x1.40mm_HandSolder, symbol Device:R
- H1, H2, H3, H4: footprint MountingHole:MountingHole_3.2mm_M3 -> MountingHole:MountingHole_3.2mm_M3_Pad_Via
- Q1: footprint TO254P1040X460X1935-3:TO254P1040X460X1935-3 -> kicad-footprints-master:MOSFET_Down
Connections:
- net +24V: now also R7.1
- net 5V_4A: now also C11.2, J10.1
- net GND: now also C10.1, Q2.3 (S); no longer D1.1 (K), S1.3
- net ISO_GND_5V: now also C11.1, C12.1
- net safe-V24: now also D1.1 (K), Q2.1 (D), R7.2
- net drain: now reaches Q1.2 (G), S1.2
- net drain: now also Q2.2 (G)
- new net: C10.2, S1.3
- new net: C12.2, J10.2
Changed lines of the file:
@@
-$EndComp
-$Comp
-L Mechanical:MountingHole_Pad H21
-U 1 1 5CB718C4
-P 8800 2000
-F 0 "H21" H 8900 2049 50  0000 L CNN
-F 1 "MountingHole_Pad" H 8900 1958 50  0000 L CNN
-F 2 "TestPoint:TestPoint_THTPad_D3.0mm_Drill1.5mm" H 8800 2000 50  0001 C CNN
-F 3 "~" H 8800 2000 50  0001 C CNN
-	1    8800 2000
-	1    0    0    -1
-$EndComp
-$Comp
-L Mechanical:MountingHole_Pad H22
-U 1 1 5CB71F6F
-P 8800 2650
-F 0 "H22" H 8900 2699 50  0000 L CNN
-F 1 "MountingHole_Pad" H 8900 2608 50  0000 L CNN
-F 2 "TestPoint:TestPoint_THTPad_D3.0mm_Drill1.5mm" H 8800 2650 50  0001 C CNN
-F 3 "~" H 8800 2650 50  0001 C CNN
-	1    8800 2650
-	1    0    0    -1
 $EndComp
 $Comp
@@
 Wire Wire Line
 	2200 3900 2200 3750
-$Comp
-L Transistor_FET:IRF6711S Q1
-U 1 1 5CB747EA
-P 2900 3700
-F 0 "Q1" H 3106 3746 50  0000 L CNN
-F 1 "STP160N3LL" H 3106 3655 50  0000 L CNN
-F 2 "TO254P1040X460X1935-3:TO254P1040X460X1935-3" H 2900 3700 50  0001 C CIN
-F 3 "https://www.infineon.com/dgdl/irf6711spbf.pdf?fileId=5546d462533600a4015355ecec0b1a7a" H 2900 3700 50  0001 L CNN
-	1    2900 3700
-	1    0    0    -1
-$EndComp
 Wire Wire Line
 	2200 2400 2200 2250
-Text GLabel 3000 3050 1    50   Input ~ 0
+Text GLabel 3000 3300 1    50   Input ~ 0
 safe-V24
 Text GLabel 1200 7000 3    50   Input ~ 0
@@
 	1    0    0    -1
 $EndComp
-Text GLabel 8800 2100 3    50   Input ~ 0
-5V_4A
 Text GLabel 5400 4350 3    50   Input ~ 0
-ISO_GND_5V
-Text GLabel 8800 2750 3    50   Input ~ 0
 ISO_GND_5V
 Text GLabel 6400 4350 3    50   Input ~ 0
@@
 F 0 "H1" H 8350 4696 50  0000 L CNN
 F 1 "MountingHole" H 8350 4605 50  0000 L CNN
-F 2 "MountingHole:MountingHole_3.2mm_M3" H 8250 4650 50  0001 C CNN
+F 2 "MountingHole:MountingHole_3.2mm_M3_Pad_Via" H 8250 4650 50  0001 C CNN
 F 3 "~" H 8250 4650 50  0001 C CNN
 	1    8250 4650
@@
 F 0 "H3" H 8950 4596 50  0000 L CNN
 F 1 "MountingHole" H 8950 4505 50  0000 L CNN
-F 2 "MountingHole:MountingHole_3.2mm_M3" H 8850 4550 50  0001 C CNN
+F 2 "MountingHole:MountingHole_3.2mm_M3_Pad_Via" H 8850 4550 50  0001 C CNN
 F 3 "~" H 8850 4550 50  0001 C CNN
 	1    8850 4550
@@
 F 0 "H2" H 8500 5096 50  0000 L CNN
 F 1 "MountingHole" H 8500 5005 50  0000 L CNN
-F 2 "MountingHole:MountingHole_3.2mm_M3" H 8400 5050 50  0001 C CNN
+F 2 "MountingHole:MountingHole_3.2mm_M3_Pad_Via" H 8400 5050 50  0001 C CNN
 F 3 "~" H 8400 5050 50  0001 C CNN
 	1    8400 5050
@@
 F 0 "H4" H 9200 5046 50  0000 L CNN
 F 1 "MountingHole" H 9200 4955 50  0000 L CNN
-F 2 "MountingHole:MountingHole_3.2mm_M3" H 9100 5000 50  0001 C CNN
+F 2 "MountingHole:MountingHole_3.2mm_M3_Pad_Via" H 9100 5000 50  0001 C CNN
 F 3 "~" H 9100 5000 50  0001 C CNN
 	1    9100 5000
@@
 	1    1600 4650
 	1    0    0    -1
-$EndComp
-$Comp
-L power:GND #PWR0114
-U 1 1 5CB988C7
-P 1250 4650
-F 0 "#PWR0114" H 1250 4400 50  0001 C CNN
-F 1 "GND" V 1255 4522 50  0000 R CNN
-F 2 "" H 1250 4650 50  0001 C CNN
-F 3 "" H 1250 4650 50  0001 C CNN
-	1    1250 4650
-	0    1    1    0
 $EndComp
 $Comp
@@
 L power:GND #PWR0116
 U 1 1 5CC0A55C
-P 2550 2650
-F 0 "#PWR0116" H 2550 2400 50  0001 C CNN
-F 1 "GND" H 2555 2477 50  0000 C CNN
-F 2 "" H 2550 2650 50  0001 C CNN
-F 3 "" H 2550 2650 50  0001 C CNN
-	1    2550 2650
+P 2550 2200
+F 0 "#PWR0116" H 2550 1950 50  0001 C CNN
+F 1 "GND" H 2555 2027 50  0000 C CNN
+F 2 "" H 2550 2200 50  0001 C CNN
+F 3 "" H 2550 2200 50  0001 C CNN
+	1    2550 2200
 	-1   0    0    1
 $EndComp
@@
 Wire Wire Line
 	2700 2850 2650 2850
-Wire Wire Line
-	2700 2850 2700 3700
-Wire Wire Line
-	3000 3050 3000 3500
 $Comp
 L Device:LED D2
@@
 Text GLabel 2200 5200 2    50   Input ~ 0
 5V_4A
+Text GLabel 1250 4650 0    50   Input ~ 0
+safe-V24
+Text GLabel 3950 3300 1    50   Input ~ 0
+safe-V24
+$Comp
+L Transistor_FET:IRF6711S Q2
+U 1 1 5CD03FA1
+P 3850 3700
+F 0 "Q2" H 4056 3746 50  0000 L CNN
+F 1 "STP160N3LL" H 4056 3655 50  0000 L CNN
+F 2 "kicad-footprints-master:MOSFET_Down" H 3850 3700 50  0001 C CIN
+F 3 "https://www.infineon.com/dgdl/irf6711spbf.pdf?fileId=5546d462533600a4015355ecec0b1a7a" H 3850 3700 50  0001 L CNN
+	1    3850 3700
+	1    0    0    -1
+$EndComp
+$Comp
+L Transistor_FET:IRF6711S Q1
+U 1 1 5CB747EA
+P 2900 3700
+F 0 "Q1" H 3106 3746 50  0000 L CNN
+F 1 "STP160N3LL" H 3106 3655 50  0000 L CNN
+F 2 "kicad-footprints-master:MOSFET_Down" H 2900 3700 50  0001 C CIN
+F 3 "https://www.infineon.com/dgdl/irf6711spbf.pdf?fileId=5546d462533600a4015355ecec0b1a7a" H 2900 3700 50  0001 L CNN
+	1    2900 3700
+	1    0    0    -1
+$EndComp
+Text Label 2700 3700 2    50   ~ 0
+drain
+Text Label 2700 2850 3    50   ~ 0
+drain
+Text Label 3650 3700 1    50   ~ 0
+drain
+Wire Wire Line
+	3950 3900 3000 3900
+Connection ~ 3000 3900
+$Comp
+L Device:R R7
+U 1 1 5CD1291C
+P 5150 2150
+F 0 "R7" H 5220 2196 50  0000 L CNN
+F 1 "R" H 5220 2105 50  0000 L CNN
+F 2 "Resistor_SMD:R_0805_2012Metric_Pad1.15x1.40mm_HandSolder" V 5080 2150 50  0001 C CNN
+F 3 "~" H 5150 2150 50  0001 C CNN
+	1    5150 2150
+	1    0    0    -1
+$EndComp
+Wire Wire Line
+	5150 2000 4650 2000
+Connection ~ 4650 2000
+Wire Wire Line
+	5150 2300 4650 2300
+Connection ~ 4650 2300
+$Comp
+L Connector:Barrel_Jack J10
+U 1 1 5CD159EA
+P 7800 2550
+F 0 "J10" H 7857 2875 50  0000 C CNN
+F 1 "Barrel_Jack" H 7857 2784 50  0000 C CNN
+F 2 "Connector_BarrelJack:BarrelJack_CUI_PJ-063AH_Horizontal" H 7850 2510 50  0001 C CNN
+F 3 "~" H 7850 2510 50  0001 C CNN
+	1    7800 2550
+	1    0    0    -1
+$EndComp
+Text GLabel 8650 2650 2    50   Input ~ 0
+ISO_GND_5V
+Text GLabel 8450 2450 2    50   Input ~ 0
+5V_4A
+Text GLabel 8300 1950 1    50   Input ~ 0
+ISO_GND_5V
+$Comp
+L Device:C C10
+U 1 1 5CD6EE7E
+P 2550 2500
+F 0 "C10" H 2665 2546 50  0000 L CNN
+F 1 "3UF" H 2665 2455 50  0000 L CNN
+F 2 "Capacitor_SMD:C_0805_2012Metric_Pad1.15x1.40mm_HandSolder" H 2588 2350 50  0001 C CNN
+F 3 "~" H 2550 2500 50  0001 C CNN
+	1    2550 2500
+	1    0    0    -1
+$EndComp
+Wire Wire Line
+	2550 2350 2550 2200
+Wire Wire Line
+	8100 2450 8300 2450
+$Comp
+L Device:C C11
+U 1 1 5CD77EE2
+P 8300 2150
+F 0 "C11" H 8415 2196 50  0000 L CNN
+F 1 "3UF" H 8415 2105 50  0000 L CNN
+F 2 "Capacitor_SMD:C_0805_2012Metric_Pad1.15x1.40mm_HandSolder" H 8338 2000 50  0001 C CNN
+F 3 "~" H 8300 2150 50  0001 C CNN
+	1    8300 2150
+	1    0    0    -1
+$EndComp
+Wire Wire Line
+	8300 2000 8300 1950
+Wire Wire Line
+	8300 2300 8300 2450
+Connection ~ 8300 2450
+Wire Wire Line
+	8300 2450 8450 2450
+$Comp
+L Device:C C12
+U 1 1 5CD7B2F4
+P 8350 2650
+F 0 "C12" H 8465 2696 50  0000 L CNN
+F 1 "3UF" H 8465 2605 50  0000 L CNN
+F 2 "Capacitor_SMD:C_0805_2012Metric_Pad1.15x1.40mm_HandSolder" H 8388 2500 50  0001 C CNN
+F 3 "~" H 8350 2650 50  0001 C CNN
+	1    8350 2650
+	0    1    1    0
+$EndComp
+Wire Wire Line
+	8100 2650 8200 2650
+Wire Wire Line
+	8500 2650 8650 2650
+Wire Wire Line
+	3000 3500 3000 3300
+Wire Wire Line
+	3950 3500 3950 3300
 $EndSCHEMATC
